File: WaterDetector.brd (EAGLE design)
At the start: 25 x 25 mm, 7 parts

Commit message: Water detect board V1.00 as sent to DirtyPCBs
Parts:
- added C3: 0.1uF, SparkFun-Capacitors:0805
- added D1: MBRA140, SparkFun-DiscreteSemi:SMA-DIODE
- added Q1: (no value), SparkFun-DiscreteSemi:SOT23-3
- added R1: 1k, SparkFun-Resistors:1206
- added R2: 1M, SparkFun-Resistors:1206
- added SG1: BUZZERNS, SparkFun-Electromechanical:BUZZER-12MM-NS
- moved C2 11.3 mm to (9.53, 16.2), turned to 180 degrees
- moved C1 1.62 mm to (3.17, 18.1), turned to 180 degrees
Connections:
- removed net SENSE2: JP3.2, JP3.4, JP3.6, JP4.2, JP4.4, JP4.6
- new net N$2: Q1.1, R1.2
- new net ROLL4SENSE: JP1.6
- net 3.3V: now also D1.C, JP3.2, JP3.4, JP3.6, JP4.2, JP4.4, JP4.6, SG1.+
- net GND: now also C3.1, Q1.2, R2.1
- net SENSE: now also C3.2, R1.1, R2.2
- net WATERSENSE: now also D1.A, JP2.6, Q1.3, SG1.-; no longer JP1.6
Routing:
- net 3.3V: track 26.6 -> 71.6 mm, vias 1 -> 4
- net SENSE2: track 36.1 -> 0.00 mm, vias 3 -> 0
- net WATERSENSE: track 0.00 -> 28.8 mm
- net GND: track 1.67 -> 27.9 mm, vias 1 -> 3
- net SENSE: track 34.3 -> 45.5 mm
- net N$2: track 0.00 -> 2.68 mm
Other:
- board text added: "Loo Roll Monitor Water Detect V1.00"
- board text added: "S.Harrison 18 April 2016"
