File: WaterDetector.sch (EAGLE design)
At the start: 7 parts

Commit message: Water detect board V1.00 as sent to DirtyPCBs
Parts:
- added C3: 0.1uF, SparkFun-Capacitors:CAP0805
- added D1: MBRA140, SparkFun-DiscreteSemi:MBRA140
- added Q1: (no value), SparkFun-DiscreteSemi:TRANSISTOR_NPNSOT23-3
- added R1: 1k, SparkFun-Resistors:RESISTOR1206
- added R2: 1M, SparkFun-Resistors:RESISTOR1206
- added SG1: BUZZERNS, SparkFun-Electromechanical:BUZZERNS
Connections:
- removed net SENSE2: JP3.2, JP3.4, JP3.6, JP4.2, JP4.4, JP4.6
- new net N$2: Q1.B, R1.2
- new net ROLL4SENSE: JP1.6
- net 3.3V: now also D1.C, JP3.2, JP3.4, JP3.6, JP4.2, JP4.4, JP4.6, SG1.1
- net GND: now also C3.1, Q1.E, R2.1
- net SENSE: now also C3.2, R1.1, R2.2
- net WATERSENSE: now also D1.A, JP2.6, Q1.C, SG1.2; no longer JP1.6
Other:
- moved on the sheet: C1, C2
